Commit message: add highbay sim

File: src/gem_simulator/gem_description/urdf/gem.urdf.xacro (robot description, xacro)
@@ -1,11 +1,21 @@
 <?xml version="1.0"?>
 <robot name="gem" xmlns:xacro="http://www.ros.org/wiki/xacro">
+  <xacro:property name="steer_angle" value="0.61"/>
+  <xacro:property name="PI" value="3.1415926835897931"/>
+  <xacro:property name="tyre_length" value="0.16"/>
+  <xacro:property name="tyre_radius" value="0.295"/>
+  <xacro:arg name="velodyne_points" default="false"/>
+  <xacro:arg name="laser_points" default="false"/>
+  <xacro:property name="velodyne_points" value="$(arg velodyne_points)"/>
+  <xacro:property name="laser_points" value="$(arg laser_points)"/>
   <xacro:include filename="$(find gem_description)/urdf/gem.gazebo" />
   <xacro:include filename="$(find gem_description)/urdf/materials.xacro" />
   <xacro:include filename="$(find gem_description)/urdf/macros.xacro" />
   <xacro:include filename="$(find velodyne_description)/urdf/VLP-16.urdf.xacro"/>
+  <!-- *************************** Base link below *************************** -->
   <link name="base_footprint">
   </link>
   <link name="base_link">
+    <!--
     <inertial>
       <origin xyz="0.0410109641324594 0.000349767124208047 0.219524161679779" rpy="0 0 0" />
@@ -19,4 +29,16 @@
         izz="482.316418870047" />
     </inertial>
+    -->
+    <inertial>
+      <origin xyz="0 0 0" rpy="0 0 0" />
+      <mass value="686" />
+      <inertia
+        ixx="325"
+        ixy="0"
+        ixz="0"
+        iyy="597"
+        iyz="0"
+        izz="465" />
+    </inertial>
     <visual>
       <origin xyz="0 0 0" rpy="0 0 0" />
@@ -41,13 +63,13 @@
   <link name="chair_link">
     <inertial>
-      <origin xyz="-0.25168177279603 0.000276944933646828 0.46906166648726" rpy="0 0 0" />
-      <mass value="66.2564411399325" />
-      <inertia
-        ixx="14.0051678459864"
-        ixy="-0.00120200191290221"
-        ixz="1.77455776912037"
-        iyy="7.60803819714354"
-        iyz="0.000593044825837774"
-        izz="9.70729216894754" />
+      <origin xyz="0 0 0" rpy="0 0 0" />
+      <mass value="0" />
+      <inertia
+        ixx="0"
+        ixy="0"
+        ixz="0"
+        iyy="0"
+        iyz="0"
+        izz="0" />
     </inertial>
     <visual>
@@ -73,13 +95,13 @@
   <link name="door_link">
     <inertial>
-      <origin xyz="0.00621903196002507 5.84652914581429E-07 0.358550118826029" rpy="0 0 0" />
-      <mass value="62.4925124039456" />
-      <inertia
-        ixx="27.8360789144871"
-        ixy="1.83479416068222E-05"
-        ixz="0.311750082296841"
-        iyy="7.554911896405"
-        iyz="-2.52231014544191E-05"
-        izz="26.8975099460351" />
+      <origin xyz="0 0 0" rpy="0 0 0" />
+      <mass value="0" />
+      <inertia
+        ixx="0"
+        ixy="0"
+        ixz="0"
+        iyy="0"
+        iyz="0"
+        izz="0" />
     </inertial>
     <visual>
@@ -105,13 +127,13 @@
   <link name="top_rack_link">
     <inertial>
-      <origin xyz="0.169 0.0522767054778464 -0.657500000000002" rpy="0 0 0" />
-      <mass value="8.88367739999998" />
-      <inertia
-        ixx="1.60728217120871"
-        ixy="6.00084366111482E-18"
-        ixz="-9.81342263314531E-17"
-        iyy="1.72456661616785"
-        iyz="-5.92489168501132E-16"
-        izz="0.152983311828453" />
+      <origin xyz="0 0 0" rpy="0 0 0" />
+      <mass value="0" />
+      <inertia
+        ixx="0"
+        ixy="0"
+        ixz="0"
+        iyy="0"
+        iyz="0"
+        izz="0" />
     </inertial>
     <visual>
@@ -137,13 +159,13 @@
   <link name="front_rack_link">
     <inertial>
-      <origin xyz="6.075819031226E-08 0.307874350591294 0.0128881009983504" rpy="0 0 0" />
-      <mass value="2.56587584103832" />
-      <inertia
-        ixx="0.0399935403341327"
-        ixy="3.94985201351379E-09"
-        ixz="4.81783258455845E-09"
-        iyy="0.17153401949232"
-        iyz="-0.00251237710479529"
-        izz="0.207040614168028" />
+      <origin xyz="0 0 0" rpy="0 0 0" />
+      <mass value="0" />
+      <inertia
+        ixx="0."
+        ixy="0"
+        ixz="0"
+        iyy="0"
+        iyz="0"
+        izz="0" />
     </inertial>
     <visual>
@@ -169,13 +191,13 @@
   <link name="rear_rack_link">
     <inertial>
-      <origin xyz="6.1506188045457E-08 0.310150326128451 0.0147333533268064" rpy="0 0 0" />
-      <mass value="2.53467167075235" />
-      <inertia
-        ixx="0.0382035938045769"
-        ixy="4.30467478765709E-09"
-        ixz="5.10550487033654E-09"
-        iyy="0.170120841320212"
-        iyz="-0.00163705466710053"
-        izz="0.205257577869692" />
+      <origin xyz="0 0 0" rpy="0 0 0" />
+      <mass value="0" />
+      <inertia
+        ixx="0"
+        ixy="0"
+        ixz="0"
+        iyy="0"
+        iyz="0"
+        izz="0" />
     </inertial>
     <visual>
@@ -201,13 +223,13 @@
   <link name="front_right_head_light_link">
     <inertial>
-      <origin xyz="0.0181463762919891 5.55111512312578E-17 3.5527136788005E-15" rpy="0 0 0" />
-      <mass value="0.269468017191218" />
-      <inertia
-        ixx="0.000596868390925667"
-        ixy="-4.5493541174505E-37"
-        ixz="-8.43232887809658E-21"
-        iyy="0.000330811799186419"
-        iyz="2.38964055770904E-36"
-        izz="0.00033081179918642" />
+      <origin xyz="0 0 0" rpy="0 0 0" />
+      <mass value="0" />
+      <inertia
+        ixx="0"
+        ixy="0"
+        ixz="0"
+        iyy="0"
+        iyz="0"
+        izz="0" />
     </inertial>
     <visual>
@@ -233,13 +255,13 @@
   <link name="front_left_head_light_link">
     <inertial>
-      <origin xyz="0.0181463762919891 -1.11022302462516E-16 3.99680288865056E-15" rpy="0 0 0" />
-      <mass value="0.269468017191218" />
-      <inertia
-        ixx="0.000596868390925667"
-        ixy="-4.5493541174505E-37"
-        ixz="-8.43232887809658E-21"
-        iyy="0.000330811799186419"
-        iyz="2.38964055770904E-36"
-        izz="0.00033081179918642" />
+      <origin xyz="0 0 0" rpy="0 0 0" />
+      <mass value="0" />
+      <inertia
+        ixx="0"
+        ixy="0"
+        ixz="0"
+        iyy="0"
+        iyz="0"
+        izz="0" />
     </inertial>
     <visual>
@@ -265,13 +287,13 @@
   <link name="front_right_turn_light_link">
     <inertial>
-      <origin xyz="0.0135004225053658 0 3.99680288865056E-15" rpy="0 0 0" />
-      <mass value="0.065815901054829" />
-      <inertia
-        ixx="4.78304226243906E-05"
-        ixy="-4.43957359734856E-38"
-        ixz="6.07038039167315E-22"
-        iyy="2.82661732953809E-05"
-        iyz="1.76248991828734E-37"
-        izz="2.82661732953809E-05" />
+      <origin xyz="0 0 0" rpy="0 0 0" />
+      <mass value="0" />
+      <inertia
+        ixx="0"
+        ixy="0"
+        ixz="0"
+        iyy="0"
+        iyz="0"
+        izz="0" />
     </inertial>
     <visual>
@@ -297,13 +319,13 @@
   <link name="front_left_turn_light_link">
     <inertial>
-      <origin xyz="0.0135004225053658 0 3.99680288865056E-15" rpy="0 0 0" />
-      <mass value="0.065815901054829" />
-      <inertia
-        ixx="4.78304226243906E-05"
-        ixy="-4.43957359734856E-38"
-        ixz="6.07038039167315E-22"
-        iyy="2.82661732953809E-05"
-        iyz="1.76248991828734E-37"
-        izz="2.82661732953809E-05" />
+      <origin xyz="0 0 0" rpy="0 0 0" />
+      <mass value="0" />
+      <inertia
+        ixx="0"
+        ixy="0"
+        ixz="0"
+        iyy="0"
+        iyz="0"
+        izz="0" />
     </inertial>
     <visual>
@@ -329,13 +351,13 @@
   <link name="rear_right_light_link">
     <inertial>
-      <origin xyz="-0.00499999999999989 -2.77555756156289E-17 -9.76996261670138E-15" rpy="0 0 0" />
-      <mass value="0.0318086256175967" />
-      <inertia
-        ixx="3.22062334378166E-05"
-        ixy="-1.38305597517403E-38"
-        ixz="6.87334333960818E-36"
-        iyy="1.6368188599055E-05"
-        iyz="-1.39682298768093E-51"
-        izz="1.6368188599055E-05" />
+      <origin xyz="0 0 0" rpy="0 0 0" />
+      <mass value="0" />
+      <inertia
+        ixx="0"
+        ixy="0"
+        ixz="0"
+        iyy="0"
+        iyz="0"
+        izz="0" />
     </inertial>
     <visual>
@@ -361,13 +383,13 @@
   <link name="rear_left_light_link">
     <inertial>
-      <origin xyz="-0.00499999999999989 0 -1.02140518265514E-14" rpy="0 0 0" />
-      <mass value="0.0318086256175967" />
-      <inertia
-        ixx="3.22062334378166E-05"
-        ixy="-1.38305597517403E-38"
-        ixz="6.87334333960818E-36"
-        iyy="1.6368188599055E-05"
-        iyz="-1.39682298768093E-51"
-        izz="1.6368188599055E-05" />
+      <origin xyz="0 0 0" rpy="0 0 0" />
+      <mass value="0" />
+      <inertia
+        ixx="0"
+        ixy="0"
+        ixz="0"
+        iyy="0"
+        iyz="0"
+        izz="0" />
     </inertial>
     <visual>
@@ -393,13 +415,13 @@
   <link name="rear_left_stop_light_link">
     <inertial>
-      <origin xyz="0.00972430253262702 9.82547376793264E-15 -9.32587340685131E-15" rpy="0 0 0" />
-      <mass value="0.109202778987047" />
-      <inertia
-        ixx="0.000190538645890679"
-        ixy="6.45440196434648E-19"
-        ixz="-3.41278961232262E-21"
-        iyy="9.87843441608066E-05"
-        iyz="-9.37294393995117E-36"
-        izz="9.87843441608066E-05" />
+      <origin xyz="0 0 0" rpy="0 0 0" />
+      <mass value="0" />
+      <inertia
+        ixx="0"
+        ixy="0"
+        ixz="0"
+        iyy="0"
+        iyz="0"
+        izz="0" />
     </inertial>
     <visual>
@@ -425,13 +447,13 @@
   <link name="rear_right_stop_light_link">
     <inertial>
-      <origin xyz="0.00972430253262724 9.82547376793264E-15 -1.02140518265514E-14" rpy="0 0 0" />
-      <mass value="0.109202778987047" />
-      <inertia
-        ixx="0.000190538645890679"
-        ixy="6.45440196434648E-19"
-        ixz="-3.41278961232262E-21"
-        iyy="9.87843441608066E-05"
-        iyz="-9.37294393995117E-36"
-        izz="9.87843441608066E-05" />
+      <origin xyz="0 0 0" rpy="0 0 0" />
+      <mass value="0" />
+      <inertia
+        ixx="0"
+        ixy="0"
+        ixz="0"
+        iyy="0"
+        iyz="0"
+        izz="0" />
     </inertial>
     <visual>
@@ -457,13 +479,13 @@
   <link name="right_blue_outer_link">
     <inertial>
-      <origin xyz="-5.55111512312578E-17 0.005 0" rpy="0 0 0" />
-      <mass value="0.104700000000001" />
-      <inertia
-        ixx="0.00181327500000001"
-        ixy="-5.27013311869779E-23"
-        ixz="-2.77932685817817E-19"
-        iyy="0.00257909140000001"
-        iyz="-1.43496084528411E-21"
-        izz="0.000767561400000003" />
+      <origin xyz="0 0 0" rpy="0 0 0" />
+      <mass value="0" />
+      <inertia
+        ixx="0"
+        ixy="0"
+        ixz="0"
+        iyy="0"
+        iyz="0"
+        izz="0" />
     </inertial>
     <visual>
@@ -489,13 +511,13 @@
   <link name="right_I_link">
     <inertial>
-      <origin xyz="-5.55111512312578E-17 0.005 4.44089209850063E-16" rpy="0 0 0" />
-      <mass value="0.266" />
-      <inertia
-        ixx="0.00324508333333333"
-        ixy="2.86326238812301E-21"
-        ixz="-9.03626747764308E-20"
-        iyy="0.00398107733333333"
-        iyz="-3.62249939950654E-37"
-        izz="0.000740427333333333" />
+      <origin xyz="0 0 0" rpy="0 0 0" />
+      <mass value="0" />
+      <inertia
+        ixx="0"
+        ixy="0"
+        ixz="0"
+        iyy="0"
+        iyz="0"
+        izz="0" />
     </inertial>
     <visual>
@@ -521,13 +543,13 @@
   <link name="left_blue_outer_link">
     <inertial>
-      <origin xyz="-5.55111512312578E-17 0.00500000000000012 0" rpy="0 0 0" />
-      <mass value="0.1047" />
-      <inertia
-        ixx="0.00181327500000001"
-        ixy="9.72940865559704E-23"
-        ixz="-1.45583787809333E-19"
-        iyy="0.00257909140000001"
-        iyz="-1.84855115156062E-21"
-        izz="0.000767561400000003" />
+      <origin xyz="0 0 0" rpy="0 0 0" />
+      <mass value="0" />
+      <inertia
+        ixx="0"
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